File: PCB Design Files/MCU_Interface.kicad_sch (KiCad schematic)
At the start: 35 parts, among them J301 UART_Header, J302 SWD_Header, SW301 RST, SW302 On/Off, SW303 Slew Rate, SW304 Encoder/Range Select, U301 STM32L041F6Px, U302 MCP1501, U303 AD5452YRM

Commit message: Finished board layout
Parts:
- added TP302: (no value), symbol Connector:TestPoint
- SW301: footprint irex_Button_Switch_SMD:SW_PUSH-12mm_Wuerth-430476085716_HandSolder -> irex_Button_Switch_SMD:SW-PUSH-6x3.5mm_CK-PTS636SL43x_HandSolder
Connections:
- net DAC_OUT_UNBUFFERED: now also TP302.1
Changed lines of the file:
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@@
   (junction (at 261.62 121.92) (diameter 0) (color 0 0 0 0)
+  )
+  (junction (at 278.13 240.03) (diameter 0) (color 0 0 0 0)
   )
   (junction (at 48.26 34.29) (diameter 0) (color 0 0 0 0)
@@
     (stroke (width 0) (type default) (color 0 0 0 0))
   )
-  (wire (pts (xy 271.78 240.03) (xy 279.4 240.03))
+  (wire (pts (xy 278.13 236.22) (xy 278.13 240.03))
+    (stroke (width 0) (type default) (color 0 0 0 0))
+  )
+  (wire (pts (xy 271.78 240.03) (xy 278.13 240.03))
     (stroke (width 0) (type default) (color 0 0 0 0))
   )
@@
   )
   (wire (pts (xy 115.57 163.83) (xy 115.57 166.37))
+    (stroke (width 0) (type default) (color 0 0 0 0))
+  )
+  (wire (pts (xy 278.13 240.03) (xy 285.75 240.03))
     (stroke (width 0) (type default) (color 0 0 0 0))
   )
@@
     (effects (font (size 1.27 1.27)) (justify left))
   )
-  (hierarchical_label "DAC_OUT_UNBUFFERED" (shape output) (at 279.4 240.03 0)
+  (hierarchical_label "DAC_OUT_UNBUFFERED" (shape output) (at 285.75 240.03 0)
     (effects (font (size 1.27 1.27)) (justify left))
   )
@@
       (effects (font (size 1.27 1.27)) (justify right))
     )
-    (property "Footprint" "irex_Button_Switch_SMD:SW_PUSH-12mm_Wuerth-430476085716_HandSolder" (id 2) (at 31.75 207.01 0)
+    (property "Footprint" "irex_Button_Switch_SMD:SW-PUSH-6x3.5mm_CK-PTS636SL43x_HandSolder" (id 2) (at 31.75 207.01 0)
       (effects (font (size 1.27 1.27)) hide)
     )
@@
     )
     (property "Datasheet" "" (id 3) (at 99.06 166.37 0)
+      (effects (font (size 1.27 1.27)) hide)
+    )
+    (pin "1")
+  )
+  (symbol (lib_id "Connector:TestPoint") (at 278.13 236.22 0) (unit 1)
+    (in_bom yes) (on_board yes) (fields_autoplaced)
+    (property "Reference" "TP302" (id 0) (at 279.527 232.0833 0)
+      (effects (font (size 1.27 1.27)) (justify left))
+    )
+    (property "Value" "" (id 1) (at 279.527 234.6202 0)
+      (effects (font (size 1.27 1.27)) (justify left))
+    )
+    (property "Footprint" "" (id 2) (at 283.21 236.22 0)
+      (effects (font (size 1.27 1.27)) hide)
+    )
+    (property "Datasheet" "~" (id 3) (at 283.21 236.22 0)
       (effects (font (size 1.27 1.27)) hide)
     )
@@
       (effects (font (size 1.27 1.27)) hide)
     )
-    (property "Value" "" (id 1) (at 264.16 186.9242 0))
+    (property "Value" "PWR_FLAG" (id 1) (at 264.16 186.9242 0))
     (property "Footprint" "" (id 2) (at 264.16 190.5 0)
       (effects (font (size 1.27 1.27)) hide)

Commit message: Added fan shroud 3D model and heatsink drawing
Parts:
- TP302: value (none) -> TestPoint; footprint (none) -> TestPoint:TestPoint_THTPad_D2.5mm_Drill1.2mm
Changed lines of the file:
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@@
       (effects (font (size 1.27 1.27)) (justify left))
     )
-    (property "Value" "" (id 1) (at 279.527 234.6202 0)
+    (property "Value" "TestPoint" (id 1) (at 279.527 234.6202 0)
       (effects (font (size 1.27 1.27)) (justify left))
     )
-    (property "Footprint" "" (id 2) (at 283.21 236.22 0)
+    (property "Footprint" "TestPoint:TestPoint_THTPad_D2.5mm_Drill1.2mm" (id 2) (at 283.21 236.22 0)
       (effects (font (size 1.27 1.27)) hide)
     )
