File: PCB Design Files/Ampeater.kicad_sch (KiCad schematic)
At the start: 17 parts, among them J101 12V Input, J102 I+_ThroughHole, J103 I+_Banana, J104 I_TerminalBlock, J105 I-_Banana, J106 I-_ThroughHole, SW101 Power Switch, U101 AZ1117-3.3

Commit message: Added initial prototype software
Parts:
- D101: value Pink -> (none); footprint irex_LED_SMD:LED_Kingbright_AA3528V_3.5x2.8mm_handsolder -> (none); Digi-Key PN (none) -> 754-1534-1-ND
Changed lines of the file:
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@@
       (effects (font (size 1.27 1.27)) (justify right))
     )
-    (property "Value" "Pink" (id 1) (at 91.821 52.8197 90)
+    (property "Value" "" (id 1) (at 91.821 52.8197 90)
       (effects (font (size 1.27 1.27)) (justify right))
     )
-    (property "Footprint" "irex_LED_SMD:LED_Kingbright_AA3528V_3.5x2.8mm_handsolder" (id 2) (at 88.9 49.53 0)
+    (property "Footprint" "" (id 2) (at 88.9 49.53 0)
       (effects (font (size 1.27 1.27)) hide)
     )
@@
       (effects (font (size 1.27 1.27)) hide)
     )
+    (property "Digi-Key PN" "754-1534-1-ND" (id 4) (at 88.9 49.53 0)
+      (effects (font (size 1.27 1.27)) hide)
+    )
